File: kicad/KoeBlaster/KoeBlaster.kicad_pcb (KiCad board)
At the start: 2 copper layers, 92.5 x 76 mm, 56 parts, among them IC1 74LVC2G14GV,125, J1 USB_B_Mini, J2 SJ2-25103A-SMT-TR, J3 SJ2-25103A-SMT-TR, Q1 SI9933CDY-T1-GE3, Q3 BC817DS, Q6 SQ2310CES-T1_GE3, U1 ESP32-WROOM-32, U2 CH340C, U3 NCP1117-3.3_SOT223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

Commit message: Updated hardware to v0.3
Parts:
- removed D3, D4: ESD5Z5.0T1G, Diode_SMD:D_SOD-523
- removed J3: SJ2-25103A-SMT-TR, SJ2-25103A-SMT-TR:CUI_SJ2-25103A-SMT-TR
- added C10: 1uF, Capacitor_SMD:C_0805_2012Metric_Pad1.18x1.45mm_HandSolder, F.Cu at (142.2, 61.0)
- added C11: 1uF, Capacitor_SMD:C_0805_2012Metric_Pad1.18x1.45mm_HandSolder, F.Cu at (77.1, 64.0)
- added D5: SP0502BAHT, Package_TO_SOT_SMD:SOT-23, F.Cu at (111.1, 97.2)
- added D_FRONTSMT1: SFH 4244-QR, koeblaster_devices:LED_SFH_4244-QR-Z, F.Cu at (90.8, 39.1)
- added D_FRONTSMT2: SFH 4244-QR, koeblaster_devices:LED_SFH_4244-QR-Z, F.Cu at (120.7, 39.1)
- added D_SIDESMT1: SFH 4244-QR, koeblaster_devices:LED_SFH_4244-QR-Z, F.Cu at (69.3, 69.2)
- added D_SIDESMT2: SFH 4244-QR, koeblaster_devices:LED_SFH_4244-QR-Z, F.Cu at (139.2, 69.8)
- added D_TOP2: SFH 4547, LED_THT:LED_D5.0mm_IRBlack, F.Cu at (113.4, 52.7)
- added D_TOPSMT1: SFH 4243-Q1R2, SFH_4243-Q1R2:LEDM3528X210N, F.Cu at (84.6, 68.1)
- added D_TOPSMT2: SFH 4243-Q1R2, SFH_4243-Q1R2:LEDM3528X210N, F.Cu at (112.1, 52.7)
- added G***: LOGO, LOGO, F.Cu at (143.0, 52.1)
- added Q2: SI2312CDS-T1-GE3, SamacSys_Parts:SOT95P237X112-3N, F.Cu at (85.0, 59.2)
- added R7: 10k, Resistor_SMD:R_0805_2012Metric_Pad1.20x1.40mm_HandSolder, F.Cu at (88.8, 58.2)
- added USB1: USB_B_Mini, koeblaster_devices:MICRO-USB-SMD_BTC-TC5T-23, B.Cu at (101.0, 99.5)
- C3, C4: footprint Capacitor_Tantalum_SMD:CP_EIA-2012-15_AVX-P_Pad1.30x1.05mm_HandSolder -> Capacitor_Tantalum_SMD:CP_EIA-3216-18_Kemet-A_Pad1.58x1.35mm_HandSolder
- C7: footprint Capacitor_SMD:C_0805_2012Metric_Pad1.18x1.45mm_HandSolder -> Capacitor_Tantalum_SMD:CP_EIA-3528-12_Kemet-T_Pad1.50x2.35mm_HandSolder
- D_FRONT1, D_FRONT2: moved to F.Cu
- D_SIDE1, D_SIDE2: footprint LED_THT:LED_D5.0mm_Horizontal_O3.81mm_Z3.0mm -> LED_THT:LED_D5.0mm_Horizontal_O6.35mm_Z3.0mm; moved to F.Cu
- J1: value USB_B_Mini -> PJ-2180-SMT; footprint SamacSys_Parts:629105150521 -> koeblaster_devices:PJ-2180-SMT
- J2: value SJ2-25103A-SMT-TR -> PJ-2180-SMT; footprint SJ2-25103A-SMT-TR:CUI_SJ2-25103A-SMT-TR -> koeblaster_devices:PJ-2180-SMT
- Q6: value SQ2310CES-T1_GE3 -> SI2312CDS-T1-GE3
- R10, R12, R8: value 5R -> 3R
- U3: value NCP1117-3.3_SOT223 -> NCP1117-3.3
- U4: value TSMP98100 -> TSOP58338
- moved R10 59.5 mm to (129.0, 39.2), turned to 90 degrees
- moved D_TOP1 27.5 mm to (85.9, 68.1), turned to 180 degrees
- moved R8 15.0 mm to (98.8, 39.1)
- moved J1 14.4 mm to (115.2, 102.7), turned to 93 degrees
- moved R12 13.7 mm to (90.2, 65.8), turned to -90 degrees
- moved J2 12.7 mm to (127.4, 101.6), turned to 98 degrees
- moved Q6 9.73 mm to (92.8, 54.0), turned to 90 degrees
- moved R15 6.52 mm to (88.8, 53.8), turned to 90 degrees
- moved D_SIDE1 3.38 mm to (71.7, 68.5), turned to -103 degrees
- moved D_FRONT1 3.02 mm to (92.0, 41.1), turned to 180 degrees
- moved D_SIDE2 3.01 mm to (137.8, 71.4), turned to 103 degrees
- moved D_FRONT2 2.96 mm to (122.0, 41.0), turned to 180 degrees
- moved C3 2.89 mm to (76.7, 59.6)
- moved R2 2.29 mm to (83.2, 73.7), turned to -90 degrees
- moved C5 2.16 mm to (98.4, 54.6)
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Connections:
- net /GPIO16 renamed /IR_INT_FRONT_SIDE
- D_FRONT2 pad 1: Net-(D_FRONT1-A) -> Net-(D_FRONT2-K)
- D_FRONT2 pad 2: +5V -> Net-(D_FRONT2-A)
- D_SIDE1 pad 1: Net-(D_SIDE1-K) -> Net-(D_FRONT1-A)
- D_SIDE1 pad 2: Net-(D_SIDE1-A) -> +5V
- D_SIDE2 pad 1: Net-(D_SIDE1-A) -> Net-(D_FRONT2-A)
- D_TOP1 pad 2: +5V -> Net-(D_TOP1-A)
- J1 pad 2: /UD- -> GND
- J1 pad 5: GND -> Net-(D5-K-Pad2)
- J2 pad 2: Net-(D3-K) -> GND
- R10 pad 2: Net-(D_SIDE1-K) -> Net-(D_FRONT2-K)
- R11 pad 1: Net-(D4-K) -> Net-(D5-K-Pad1)
- R12 pad 1: Net-(Q6-D) -> Net-(Q2-D)
- R9 pad 1: Net-(D3-K) -> Net-(D5-K-Pad2)
- U1 pad 13: unconnected-(U1-IO14-Pad13) -> /IR_INT_TOP
Routing:
- net Net-(D_SIDE1-A): track 112.3 -> 0.00 mm, vias 1 -> 0
- net Net-(D_FRONT2-A): track 0.00 -> 49.3 mm
- net Net-(D_TOP1-A): track 0.00 -> 40.8 mm
- net +5V: track 196.5 -> 216.4 mm, vias 5 -> 8
- net Net-(D5-K-Pad1): track 0.00 -> 19.5 mm, vias 0 -> 1
- net Net-(D_TOP1-K): track 23.6 -> 4.85 mm, vias 1 -> 0
- net /IR_INT_TOP: track 0.00 -> 15.2 mm
- net Net-(D4-K): track 14.4 -> 0.00 mm, vias 1 -> 0
- net +3V3: track 133.8 -> 120.5 mm
- net Net-(D5-K-Pad2): track 0.00 -> 12.3 mm, vias 0 -> 1
- net Net-(Q6-D): track 39.5 -> 49.5 mm, vias 4 -> 2
- net GND: track 1.47 -> 10.9 mm, vias 34 -> 43
- net /EN: track 46.8 -> 56.2 mm
- net Net-(D_SIDE1-K): track 8.89 -> 0.00 mm
- net Net-(D_FRONT2-K): track 0.00 -> 8.19 mm
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Other:
- board text added: "KoeBlaster v0.3 03/2025"
- board text removed: "KoeBlaster v0.2 04/2024"
