File: kicad/KoeBlaster/KoeBlaster.kicad_sch (KiCad schematic)
At the start: 48 parts, among them IC1 74LVC2G14GV,125, J1 USB_B_Mini, J2 SJ2-25103A-SMT-TR, J3 SJ2-25103A-SMT-TR, Q1 SI9933CDY-T1-GE3, Q3 BC817DS, Q6 SQ2310CES-T1_GE3, U1 ESP32-WROOM-32, U2 CH340C, U3 NCP1117-3.3_SOT223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

Commit message: Updated hardware to v0.3
Parts:
- removed C7: 100uF, Capacitor_SMD:C_0805_2012Metric_Pad1.18x1.45mm_HandSolder, symbol Device:C
- removed D3, D4: ESD5Z5.0T1G, Diode_SMD:D_SOD-523, symbol Diode:ESD5Zxx
- removed J1: USB_B_Mini, SamacSys_Parts:629105150521, symbol SamacSys_Parts:629105150521
- removed J2, J3: SJ2-25103A-SMT-TR, CUI_SJ2-25103A-SMT-TR, symbol koeblaster_devices:SJ2-25103A-SMT-TR
- added C10, C11: 1uF, Capacitor_SMD:C_0805_2012Metric_Pad1.18x1.45mm_HandSolder, symbol Device:C
- added C7: 100uF, Capacitor_Tantalum_SMD:CP_EIA-3528-12_Kemet-T_Pad1.50x2.35mm_HandSolder, symbol Device:C_Polarized
- added D5: SP0502BAHT, Package_TO_SOT_SMD:SOT-23, symbol Power_Protection:SP0502BAHT
- added D_FRONTSMT1, D_FRONTSMT2, D_SIDESMT1, D_SIDESMT2: SFH 4244-QR, koeblaster_devices:LED_SFH_4244-QR-Z, symbol Device:LED_Small_Filled
- added D_TOP2: SFH 4547, LED_THT:LED_D5.0mm_IRBlack, symbol Device:LED_Small_Filled
- added D_TOPSMT1, D_TOPSMT2: SFH 4243-Q1R2, SFH_4243-Q1R2:LEDM3528X210N, symbol Device:LED_Small_Filled
- added J1, J2: PJ-2180-SMT, koeblaster_devices:PJ-2180-SMT, symbol koeblaster_devices:PJ-2180-SMT
- added Q2: SI2312CDS-T1-GE3, SamacSys_Parts:SOT95P237X112-3N, symbol SamacSys_Parts:SQ2310CES-T1_GE3
- added R7: 10k, Resistor_SMD:R_0805_2012Metric_Pad1.20x1.40mm_HandSolder, symbol Device:R
- added USB1: USB_B_Mini, koeblaster_devices:MICRO-USB-SMD_BTC-TC5T-23, symbol koeblaster_devices:BTC-TC5T-23
- C3, C4: footprint Capacitor_Tantalum_SMD:CP_EIA-2012-15_AVX-P_Pad1.30x1.05mm_HandSolder -> Capacitor_Tantalum_SMD:CP_EIA-3216-18_Kemet-A_Pad1.58x1.35mm_HandSolder
- D_SIDE1, D_SIDE2: footprint LED_THT:LED_D5.0mm_Horizontal_O3.81mm_Z3.0mm -> LED_THT:LED_D5.0mm_Horizontal_O6.35mm_Z3.0mm
- H1, H2, R18, S2: now left out of the parts list
- Q6: value SQ2310CES-T1_GE3 -> SI2312CDS-T1-GE3; Manufacturer_Part_Number SQ2310CES-T1_GE3 -> SI2312CDS-T1-GE3
- R10, R12, R8: value 5R -> 3R
- U3: value NCP1117-3.3_SOT223 -> NCP1117-3.3
- U4: value TSMP98100 -> TSOP58338
Connections:
- net +3V3: now also C7.1
- net +5V: now also D_SIDE1.2 (A), C10.1, C11.1, D_SIDESMT1.2 (A), D_SIDESMT2.2 (A), D_TOP2.2 (A), D_TOPSMT2.2 (A), USB1.1 (VBUS); no longer D_FRONT2.2 (A), D_TOP1.2 (A)
- net GND: now also C10.2, C11.2, C7.2, D5.3 (A), J1.2, J2.2, Q2.2 (S), R7.2, USB1.5 (GND), USB1.6 (EP)
- net UD+: now also USB1.3 (D+)
- net UD-: now also USB1.2 (D-)
- net at R11.1: now also D5.1 (K), J2.5
- net at Q6.3 (D), R10.1, R8.1: no longer R12.1
- net at R9.1: now also D5.2 (K), J1.5
- net at D_FRONT1.1 (K), R8.2: now also D_FRONTSMT1.1 (K)
- net IR_INT_TOP: now reaches U1.13 (IO14)
- net IR_INT_TOP: now also Q2.1 (G), R7.1
- net at D_TOP1.1 (K), R12.2: now also D_TOPSMT1.1 (K)
- net at D_SIDE2.1 (K): now also D_FRONT2.2 (A), D_FRONTSMT2.2 (A), D_SIDESMT2.1 (K); no longer D_SIDE1.2 (A)
- net at R10.2: now also D_FRONT2.1 (K), D_FRONTSMT2.1 (K); no longer D_SIDE1.1 (K)
- net at D_FRONT1.2 (A): now also D_SIDE1.1 (K), D_FRONTSMT1.2 (A), D_SIDESMT1.1 (K); no longer D_FRONT2.1 (K)
- net GPIO16 renamed IR_INT_FRONT_SIDE
- new net: D_TOP1.2 (A), D_TOP2.1 (K), D_TOPSMT1.2 (A), D_TOPSMT2.1 (K)
- new net: Q2.3 (D), R12.1
Other:
- note added: "Development Reset"
- note added: "IR Learning Sensor"
- note added: "Internal & External IR Led Stabilization"
- note added: "Power Supply"
- note added: "RGB Indicator Led"
- note added: "Reset & Factory Reset Button"
- note added: "USB Serial & Programming Interface"
- note added: "Use either SMT OR THT IR Leds. Not both!"
- moved on the sheet: C9, D1, D_FRONT1, D_FRONT2, D_SIDE1, D_SIDE2, D_TOP1, IC1, Q1A, Q1B, Q3B, R10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
